File: qdrive_2axis.kicad_sch (KiCad schematic)
At the start: 5 parts

Commit message: Fixed mounting holes
Parts:
- H203, H204: footprint MountingHole:MountingHole_2.7mm_Pad_Via -> MountingHole:MountingHole_3.2mm_M3_Pad_Via
- H401: footprint MountingHole:MountingHole_2.7mm_M2.5_Pad_Via -> MountingHole:MountingHole_3.2mm_M3_Pad_Via
Changed lines of the file:
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@@
       (effects (font (size 1.27 1.27)) (justify left) hide)
     )
-    (property "Footprint" "MountingHole:MountingHole_2.7mm_Pad_Via" (at 231.14 149.86 0)
+    (property "Footprint" "MountingHole:MountingHole_3.2mm_M3_Pad_Via" (at 231.14 149.86 0)
       (effects (font (size 1.27 1.27)) hide)
     )
@@
       (effects (font (size 1.27 1.27)) (justify left) hide)
     )
-    (property "Footprint" "MountingHole:MountingHole_2.7mm_Pad_Via" (at 219.71 149.86 0)
+    (property "Footprint" "MountingHole:MountingHole_3.2mm_M3_Pad_Via" (at 219.71 149.86 0)
       (effects (font (size 1.27 1.27)) hide)
     )
@@
       (effects (font (size 1.27 1.27)) (justify left) hide)
     )
-    (property "Footprint" "MountingHole:MountingHole_2.7mm_M2.5_Pad_Via" (at 240.03 149.86 0)
+    (property "Footprint" "MountingHole:MountingHole_3.2mm_M3_Pad_Via" (at 240.03 149.86 0)
       (effects (font (size 1.27 1.27)) hide)
     )
