File: qdrive_2axis.kicad_pcb (KiCad board)
At the start: 4 copper layers, 125 x 67 mm, 254 parts, among them J201 1054500101, J202 Conn_01x05_MountingPin, J203 Screw_Terminal_01x02, J204 Conn_01x05_MountingPin, J205 Conn_01x03, J208 NC_Conn_02x03_Odd_Even, J210 NC_Conn_01x07_Female, J211 S3B-PH-SM4-TB(LF)(SN), J301 Screw_Terminal_01x01, J302 Screw_Terminal_01x01, J306 Screw_Terminal_01x01, J307 Screw_Terminal_01x01, J309 Screw_Terminal_01x01, J401 Screw_Terminal_01x01, J402 Screw_Terminal_01x01, J403 Screw_Terminal_01x01, Q201 HYG025N06LS1C2, Q202 HYG025N06LS1C2, Q301 HYG025N06LS1C2, Q302 HYG025N06LS1C2, Q303 HYG025N06LS1C2, Q304 HYG025N06LS1C2, Q305 HYG025N06LS1C2, Q306 HYG025N06LS1C2, Q307 HYG025N06LS1C2, Q308 HYG025N06LS1C2, Q309 HYG025N06LS1C2, Q310 HYG025N06LS1C2, Q311 HYG025N06LS1C2, Q312 HYG025N06LS1C2, Q401 HYG025N06LS1C2, Q402 HYG025N06LS1C2, Q403 HYG025N06LS1C2, Q404 HYG025N06LS1C2, Q405 HYG025N06LS1C2, Q406 HYG025N06LS1C2, Q407 HYG025N06LS1C2, Q408 HYG025N06LS1C2, Q409 HYG025N06LS1C2, Q410 HYG025N06LS1C2, Q411 HYG025N06LS1C2, Q412 HYG025N06LS1C2, SW201 SKRKAHE020, U201 STM32F405RGT6, U202 TJA1050T, U203 LM5109BSD, U204 LM1117-3.3, U205 NCP51460SN33T1G, U301 DRV8301DCAR, U401 DRV8301DCAR, Y201 8MHz

Commit message: Fixed mounting holes
Parts:
- H101, H102: footprint MountingHole:MountingHole_2.7mm_Pad_Via -> MountingHole:MountingHole_3.2mm_M3_Pad_Via
- H103: footprint MountingHole:MountingHole_2.7mm_M2.5_Pad_Via -> MountingHole:MountingHole_3.2mm_M3_Pad_Via
- moved R314 3.54 mm to (159.8, 152.8), turned to -90 degrees
- moved Q404 1.30 mm to (276.9, 152.7)
- moved NT404 1.00 mm to (281.3, 155.4)
- moved R402 0.94 mm to (279.0, 142.4), turned to 0 degrees
- moved Q403 0.91 mm to (276.9, 146.4)
Connections:
- net /M0_board/AVDD_M0 renamed /M0_axis/AVDD_M0
- net /M0_board/DVDD_M0 renamed /M0_axis/DVDD_M0
- net /M0_board/M0B_DC_CAL renamed /M0_axis/M0B_DC_CAL
- net /M0_board/M0B_EN_GATE renamed /M0_axis/M0B_EN_GATE
- net /M0_board/M0B_PWRGD renamed /M0_axis/M0B_PWRGD
- net /M0_board/M0B_SO1 renamed /M0_axis/M0B_SO1
- net /M0_board/M0B_SO2 renamed /M0_axis/M0B_SO2
- net /M0_board/M0B_SPI_MISO renamed /M0_axis/M0B_SPI_MISO
- net /M0_board/M0B_SPI_MOSI renamed /M0_axis/M0B_SPI_MOSI
- net /M0_board/M0B_SPI_SCK renamed /M0_axis/M0B_SPI_SCK
- net /M0_board/M0B_TEMP renamed /M0_axis/M0B_TEMP
- net /M0_board/M0B_nCS renamed /M0_axis/M0B_nCS
- net /M0_board/M0BnFAULT renamed /M0_axis/M0BnFAULT
- net /M0_board/M0BnOCTW renamed /M0_axis/M0BnOCTW
- net /M0_board/M0_GH_A renamed /M0_axis/M0_GH_A
- net /M0_board/M0_GH_B renamed /M0_axis/M0_GH_B
- net /M0_board/M0_GH_C renamed /M0_axis/M0_GH_C
- net /M0_board/M0_GL_A renamed /M0_axis/M0_GL_A
- net /M0_board/M0_GL_B renamed /M0_axis/M0_GL_B
- net /M0_board/M0_GL_C renamed /M0_axis/M0_GL_C
- net /M0_board/M0_SH_A renamed /M0_axis/M0_SH_A
- net /M0_board/M0_SH_B renamed /M0_axis/M0_SH_B
- net /M0_board/M0_SH_C renamed /M0_axis/M0_SH_C
- net /M0_board/M0_SL_A renamed /M0_axis/M0_SL_A
- net /M0_board/M0_SL_B renamed /M0_axis/M0_SL_B
- net /M0_board/M0_SL_C renamed /M0_axis/M0_SL_C
- net /M0_board/M0_SN1 renamed /M0_axis/M0_SN1
- net /M0_board/M0_SN2 renamed /M0_axis/M0_SN2
- net /M0_board/M0_SP1 renamed /M0_axis/M0_SP1
- net /M0_board/M0_SP2 renamed /M0_axis/M0_SP2
- net /M1_board/AVDD_M1 renamed /M1_axis/AVDD_M1
- net /M1_board/DVDD_M1 renamed /M1_axis/DVDD_M1
- net /M1_board/M1B_AH renamed /M1_axis/M1B_AH
- net /M1_board/M1B_AL renamed /M1_axis/M1B_AL
- net /M1_board/M1B_BH renamed /M1_axis/M1B_BH
- net /M1_board/M1B_BL renamed /M1_axis/M1B_BL
- net /M1_board/M1B_CH renamed /M1_axis/M1B_CH
- net /M1_board/M1B_CL renamed /M1_axis/M1B_CL
- net /M1_board/M1B_DC_CAL renamed /M1_axis/M1B_DC_CAL
- net /M1_board/M1B_PWRGD renamed /M1_axis/M1B_PWRGD
- net /M1_board/M1B_SO1 renamed /M1_axis/M1B_SO1
- net /M1_board/M1B_SO2 renamed /M1_axis/M1B_SO2
- net /M1_board/M1B_TEMP renamed /M1_axis/M1B_TEMP
- net /M1_board/M1B_nCS renamed /M1_axis/M1B_nCS
- net /M1_board/M1BnOCTW renamed /M1_axis/M1BnOCTW
- net /M1_board/M1_GH_A renamed /M1_axis/M1_GH_A
- net /M1_board/M1_GH_B renamed /M1_axis/M1_GH_B
- net /M1_board/M1_GH_C renamed /M1_axis/M1_GH_C
- net /M1_board/M1_GL_A renamed /M1_axis/M1_GL_A
- net /M1_board/M1_GL_B renamed /M1_axis/M1_GL_B
- net /M1_board/M1_GL_C renamed /M1_axis/M1_GL_C
- net /M1_board/M1_SH_A renamed /M1_axis/M1_SH_A
- net /M1_board/M1_SH_B renamed /M1_axis/M1_SH_B
- net /M1_board/M1_SH_C renamed /M1_axis/M1_SH_C
- net /M1_board/M1_SL_A renamed /M1_axis/M1_SL_A
- net /M1_board/M1_SL_B renamed /M1_axis/M1_SL_B
- net /M1_board/M1_SL_C renamed /M1_axis/M1_SL_C
- net /M1_board/M1_SN1 renamed /M1_axis/M1_SN1
- net /M1_board/M1_SN2 renamed /M1_axis/M1_SN2
- net /M1_board/M1_SP1 renamed /M1_axis/M1_SP1
- net /M1_board/M1_SP2 renamed /M1_axis/M1_SP2
- net /main_board/AUX_N renamed /MCU/AUX_N
- net /main_board/AUX_P renamed /MCU/AUX_P
- net /main_board/AUX_TEMP renamed /MCU/AUX_TEMP
- net /main_board/BOOT0 renamed /MCU/BOOT0
- net /main_board/BRAKE_OUT renamed /MCU/BRAKE_OUT
- net /main_board/CAN1_H renamed /MCU/CAN1_H
- net /main_board/CAN1_L renamed /MCU/CAN1_L
- net /main_board/CAN_D renamed /MCU/CAN_D
- net /main_board/CAN_R renamed /MCU/CAN_R
- net /main_board/GPIO_1 renamed /MCU/GPIO_1
- net /main_board/GPIO_2 renamed /MCU/GPIO_2
- net /main_board/GPIO_3 renamed /MCU/GPIO_3
- net /main_board/GPIO_4 renamed /MCU/GPIO_4
- net /main_board/GPIO_5 renamed /MCU/GPIO_5
- net /main_board/GPIO_6 renamed /MCU/GPIO_6
- net /main_board/GPIO_7 renamed /MCU/GPIO_7
- net /main_board/GPIO_8 renamed /MCU/GPIO_8
- net /main_board/M0_AH renamed /MCU/M0_AH
- net /main_board/M0_AL renamed /MCU/M0_AL
- net /main_board/M0_BH renamed /MCU/M0_BH
- net /main_board/M0_BL renamed /MCU/M0_BL
- net /main_board/M0_CH renamed /MCU/M0_CH
- net /main_board/M0_CL renamed /MCU/M0_CL
- net /main_board/M0_ENC_A renamed /MCU/M0_ENC_A
- net /main_board/M0_ENC_B renamed /MCU/M0_ENC_B
- net /main_board/M0_ENC_Z renamed /MCU/M0_ENC_Z
- net /main_board/M1_ENC_A renamed /MCU/M1_ENC_A
- net /main_board/M1_ENC_B renamed /MCU/M1_ENC_B
- net /main_board/M1_ENC_Z renamed /MCU/M1_ENC_Z
- net /main_board/OSC_IN renamed /MCU/OSC_IN
- net /main_board/OSC_OUT renamed /MCU/OSC_OUT
- net /main_board/SWCLK renamed /MCU/SWCLK
- net /main_board/SWDIO renamed /MCU/SWDIO
- net /main_board/USB_D+ renamed /MCU/USB_D+
- net /main_board/USB_D- renamed /MCU/USB_D-
- net /main_board/USB_V renamed /MCU/USB_V
- net /main_board/VBUS_S renamed /MCU/VBUS_S
- net /main_board/nRST renamed /MCU/nRST
Routing:
- net Net-(Q311-G): track 10.4 -> 14.7 mm
- net /M0_axis/M0_GL_C: track 44.8 -> 41.2 mm
- net /M1_axis/M1_GL_A: track 34.5 -> 33.0 mm
- net /M1_axis/M1_SL_A: track 49.3 -> 48.0 mm
- net /M1_axis/M1_SH_A: track 36.9 -> 37.6 mm
- net GVDD_M0: track 63.5 -> 64.0 mm

Commit message: Fixes
Routing:
- net /M0_axis/M0_SP2: track 17.8 -> 19.0 mm
- net /M0_axis/M0_SN2: track 18.7 -> 19.6 mm
- net /M0_axis/M0_GH_C: track 26.0 -> 26.8 mm
- net /M0_axis/M0_SL_C: track 28.7 -> 29.2 mm
